Commit message: feat: integrate Realsense sensors, YOLO object detection with ONNX Runtime, and soft end-effector support for MyCobot trajectory control.

File: src/mycobot_description/urdf/robots/mycobot_320_ur_compatible.urdf.xacro (robot description, xacro)
@@ -51,4 +51,5 @@
     <xacro:arg name="use_gazebo" default="false"/>
     <xacro:arg name="use_gripper" default="false"/>
+    <xacro:arg name="use_soft_ee" default="true"/>
     <xacro:arg name="controllers_file" default="none"/>
     <!-- World link -->
@@ -243,10 +244,12 @@
       <origin xyz="0 0 0" rpy="0 ${-pi/2.0} ${-pi/2.0}"/>
     </joint>
-    <!-- flange-tool0 fixed joint -->
-    <joint name="$(arg prefix)flange-tool0" type="fixed">
-      <parent link="$(arg prefix)flange"/>
-      <child link="$(arg prefix)tool0"/>
-      <origin xyz="0 0 0" rpy="0 0 0"/>
-    </joint>
+    <!-- flange-tool0 fixed joint - Only add if NOT using soft end effector -->
+    <xacro:unless value="$(arg use_soft_ee)">
+      <joint name="$(arg prefix)flange-tool0" type="fixed">
+        <parent link="$(arg prefix)flange"/>
+        <child link="$(arg prefix)tool0"/>
+        <origin xyz="0 0 0" rpy="0 0 0"/>
+      </joint>
+    </xacro:unless>
     <!-- Gazebo Sim ROS2 Control Plugin -->
     <xacro:include filename="$(find mycobot_description)/urdf/control/gazebo_sim_ros2_control.urdf.xacro"/>
@@ -255,4 +258,10 @@
       use_gazebo="$(arg use_gazebo)"
       controllers_file="$(arg controllers_file)"/>
+    <!-- Include Soft End Effector -->
+    <xacro:include filename="$(find mycobot_description)/urdf/mech/soft_end_effector.urdf.xacro"/>
+    <!-- Conditionally add soft end effector -->
+    <xacro:if value="$(arg use_soft_ee)">
+      <xacro:soft_end_effector parent_link="$(arg prefix)flange" prefix="$(arg prefix)"/>
+    </xacro:if>
     <!-- UR-compatible ROS2 Control Configuration -->
     <xacro:include filename="$(find mycobot_description)/urdf/control/mycobot_320_ur_ros2_control.urdf.xacro"/>
